Commit message: ROS 2 deployment and visualization pipeline for LEAP Hand

File: ros2_ws/src/leap_deployment/urdf/leap_hand.urdf (robot description, URDF)
Before this commit: robot leap_hand, 17 links, 16 joints
Links:
- removed link if_link_0
- removed link if_link_1
- removed link if_link_2
- removed link if_link_3
- removed link mf_link_0
- removed link mf_link_1
- removed link mf_link_2
- removed link mf_link_3
- removed link rf_link_0
- removed link rf_link_1
- removed link rf_link_2
- removed link rf_link_3
- removed link th_link_0
- removed link th_link_1
- removed link th_link_2
- removed link th_link_3
- added link base_link
- added link if_bs; visual mesh filename=file:///mnt/newvolume/Programming/Python/Deep_Learning/leap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
- added link if_ds; visual mesh filename=file:///mnt/newvolume/Programming/Python/Deep_Learning/leap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; visual mesh filename=file:///mnt/newvolume/Programming/Python/Deep_Learning/leap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
- added link if_md; visual mesh filename=file:///mnt/newvolume/Programming/Python/Deep_Learning/leap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
- added link if_px; visual mesh filename=file:///mnt/newvolume/Programming/Python/Deep_Learning/leap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
- added link mf_bs; visual mesh filename=file:///mnt/newvolume/Programming/Python/Deep_Learning/leap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
- added link mf_ds; visual mesh filename=file:///mnt/newvolume/Programming/Python/Deep_Learning/leap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; visual mesh filename=file:///mnt/newvolume/Programming/Python/Deep_Learning/leap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
- added link mf_md; visual mesh filename=file:///mnt/newvolume/Programming/Python/Deep_Learning/leap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
- added link mf_px; visual mesh filename=file:///mnt/newvolume/Programming/Python/Deep_Learning/leap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
- added link rf_bs; visual mesh filename=file:///mnt/newvolume/Programming/Python/Deep_Learning/leap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
- added link rf_ds; visual mesh filename=file:///mnt/newvolume/Programming/Python/Deep_Learning/leap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; visual mesh filename=file:///mnt/newvolume/Programming/Python/Deep_Learning/leap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
- added link rf_md; visual mesh filename=file:///mnt/newvolume/Programming/Python/Deep_Learning/leap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
- added link rf_px; visual mesh filename=file:///mnt/newvolume/Programming/Python/Deep_Learning/leap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
- added link table; visual box size=0.6 0.6 0.05
- added link th_bs; visual mesh filename=file:///mnt/newvolume/Programming/Python/Deep_Learning/leap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
- added link th_ds; visual mesh filename=file:///mnt/newvolume/Programming/Python/Deep_Learning/leap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; visual mesh filename=file:///mnt/newvolume/Programming/Python/Deep_Learning/leap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
- added link th_mp; visual mesh filename=file:///mnt/newvolume/Programming/Python/Deep_Learning/leap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
- added link th_px; visual mesh filename=file:///mnt/newvolume/Programming/Python/Deep_Learning/leap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
- link palm: geometry visual mesh filename=file:///mnt/newvolume/Programming/Python/Deep_Learning/leap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
Joints:
- added joint base_link_to_palm: type fixed, parent base_link, child palm, origin xyz=0 0.04 0.16 rpy=0.000000 0.000000 0.000000, axis 0 0 1
- added joint base_link_to_table: type fixed, parent base_link, child table, origin xyz=0 0 0 rpy=0.000000 0.000000 0.000000, axis 0 0 1
- joint if_dip: axis 0 1 0 -> 0 0 -1; child if_link_3 -> if_ds; origin xyz=0 0 0.04 rpy=0 0 0 -> xyz=0 -0.0361 0.0002 rpy=0.000000 0.000000 0.000000; parent if_link_2 -> if_md
- joint if_mcp: axis 0 1 0 -> 0 0 -1; child if_link_0 -> if_bs; origin xyz=-0.01 0.04 0.05 rpy=0 0 0 -> xyz=-0.007 0.023 -0.0187 rpy=1.570793 1.570790 0.000003
- joint if_pip: axis 0 1 0 -> 0 0 -1; child if_link_2 -> if_md; origin xyz=0 0 0.04 rpy=0 0 0 -> xyz=0.015 0.0143 -0.013 rpy=1.570793 -1.570790 -0.000003; parent if_link_1 -> if_px
- joint if_rot: axis 0 1 0 -> 0 0 -1; child if_link_1 -> if_px; origin xyz=0 0 0.04 rpy=0 0 0 -> xyz=-0.0122 0.0381 0.0145 rpy=-1.570790 0.000000 1.570790; parent if_link_0 -> if_bs
- joint mf_dip: axis 0 1 0 -> 0 0 -1; child mf_link_3 -> mf_ds; origin xyz=0 0 0.04 rpy=0 0 0 -> xyz=0 -0.0361 0.0002 rpy=0.000000 0.000000 0.000000; parent mf_link_2 -> mf_md
- joint mf_mcp: axis 0 1 0 -> 0 0 -1; child mf_link_0 -> mf_bs; origin xyz=-0.01 0.0 0.05 rpy=0 0 0 -> xyz=-0.0071 -0.0224 -0.0187 rpy=1.570793 1.570790 0.000003
- joint mf_pip: axis 0 1 0 -> 0 0 -1; child mf_link_2 -> mf_md; origin xyz=0 0 0.04 rpy=0 0 0 -> xyz=0.015 0.0143 -0.013 rpy=1.570793 -1.570790 -0.000003; parent mf_link_1 -> mf_px
- joint mf_rot: axis 0 1 0 -> 0 0 -1; child mf_link_1 -> mf_px; origin xyz=0 0 0.04 rpy=0 0 0 -> xyz=-0.0122 0.0381 0.0145 rpy=-1.570790 0.000000 1.570790; parent mf_link_0 -> mf_bs
- joint rf_dip: axis 0 1 0 -> 0 0 -1; child rf_link_3 -> rf_ds; origin xyz=0 0 0.04 rpy=0 0 0 -> xyz=0 -0.03609 0.0002 rpy=0.000000 0.000000 0.000000; parent rf_link_2 -> rf_md
- joint rf_mcp: axis 0 1 0 -> 0 0 -1; child rf_link_0 -> rf_bs; origin xyz=-0.01 -0.04 0.05 rpy=0 0 0 -> xyz=-0.00709 -0.0678 -0.0187 rpy=1.570793 1.570790 0.000003
- joint rf_pip: axis 0 1 0 -> 0 0 -1; child rf_link_2 -> rf_md; origin xyz=0 0 0.04 rpy=0 0 0 -> xyz=0.015 0.0143 -0.013 rpy=1.570793 -1.570790 -0.000003; parent rf_link_1 -> rf_px
- joint rf_rot: axis 0 1 0 -> 0 0 -1; child rf_link_1 -> rf_px; origin xyz=0 0 0.04 rpy=0 0 0 -> xyz=-0.0122 0.0381 0.0145 rpy=-1.570790 0.000000 1.570790; parent rf_link_0 -> rf_bs
- joint th_axl: axis 0 1 0 -> 0 0 -1; child th_link_1 -> th_bs; origin xyz=0 0 0.04 rpy=0 0 0 -> xyz=0 0.0143 -0.013 rpy=1.570793 -1.570790 -0.000003; parent th_link_0 -> th_mp
- joint th_cmc: axis 0 1 0 -> 0 0 -1; child th_link_0 -> th_mp; origin xyz=-0.05 -0.02 0.05 rpy=0 0 0 -> xyz=-0.0693 -0.0012 -0.0216 rpy=0.000000 1.570791 0.000000
- joint th_ipl: axis 0 1 0 -> 0 0 -1; child th_link_3 -> th_ds; origin xyz=0 0 0.04 rpy=0 0 0 -> xyz=0 0.0466 0.0002 rpy=0.000000 0.000000 3.141590; parent th_link_2 -> th_px
- joint th_mcp: axis 0 1 0 -> 0 0 -1; child th_link_2 -> th_px; origin xyz=0 0 0.04 rpy=0 0 0 -> xyz=0 0.0145 -0.017 rpy=-1.570791 0.000000 0.000000; parent th_link_1 -> th_bs

Commit message: fix: make all paths relative and bundle MJCF/mesh assets locally
- generate_urdf_mjcf.py: replace 4 absolute /mnt/... paths with paths
  derived from the script's own location via os.path.abspath(__file__).
  MJCF source files now expected in ./leap_hand_mjcf/ (self-contained).
  URDF mesh refs updated from file:// absolute URIs to package://
  leap_deployment/urdf/assets/ for portable RViz2 resolution.

- policy_node.py: derive _PROJECT_ROOT at runtime from __file__; venv
  site-packages path and best_model.zip path are now fully relative.

- setup.py: add urdf/assets/*.obj to data_files so colcon build
  installs mesh assets into the package share directory.

- leap_hand_mjcf/: add locally-copied MJCF XMLs and .obj meshes so the
  repo no longer depends on the sibling leap-dexterous-grasping clone.

- ros2_ws/src/leap_deployment/urdf/assets/: add mesh assets for RViz2.

File: ros2_ws/src/leap_deployment/urdf/leap_hand.urdf (robot description, URDF)
Before this commit: robot leap_grasp_scene, 19 links, 18 joints
Links:
- link if_bs: geometry visual mesh filename=package://leap_deployment/urdf/assets/base.obj
- link if_ds: geometry visual mesh filename=package://leap_deployment/urdf/assets/distal.obj; visual mesh filename=package://leap_deployment/urdf/assets/tip.obj
- link if_md: geometry visual mesh filename=package://leap_deployment/urdf/assets/medial.obj
- link if_px: geometry visual mesh filename=package://leap_deployment/urdf/assets/proximal.obj
- link mf_bs: geometry visual mesh filename=package://leap_deployment/urdf/assets/base.obj
- link mf_ds: geometry visual mesh filename=package://leap_deployment/urdf/assets/distal.obj; visual mesh filename=package://leap_deployment/urdf/assets/tip.obj
- link mf_md: geometry visual mesh filename=package://leap_deployment/urdf/assets/medial.obj
- link mf_px: geometry visual mesh filename=package://leap_deployment/urdf/assets/proximal.obj
- link palm: geometry visual mesh filename=package://leap_deployment/urdf/assets/palm_right.obj
- link rf_bs: geometry visual mesh filename=package://leap_deployment/urdf/assets/base.obj
- link rf_ds: geometry visual mesh filename=package://leap_deployment/urdf/assets/distal.obj; visual mesh filename=package://leap_deployment/urdf/assets/tip.obj
- link rf_md: geometry visual mesh filename=package://leap_deployment/urdf/assets/medial.obj
- link rf_px: geometry visual mesh filename=package://leap_deployment/urdf/assets/proximal.obj
- link th_bs: geometry visual mesh filename=package://leap_deployment/urdf/assets/thumb_base.obj
- link th_ds: geometry visual mesh filename=package://leap_deployment/urdf/assets/thumb_distal.obj; visual mesh filename=package://leap_deployment/urdf/assets/thumb_tip.obj
- link th_mp: geometry visual mesh filename=package://leap_deployment/urdf/assets/proximal.obj
- link th_px: geometry visual mesh filename=package://leap_deployment/urdf/assets/thumb_proximal.obj
